Commit message: fix the arm

File: src/robot/kim_description/urdf/kim_kardashian.urdf.xacro (robot description, xacro)
@@ -26,17 +26,30 @@
   <link name="vertical_arm">
     <visual>
-      <origin xyz="0 0 0.2" rpy="0 0 0"/> <geometry><box size="0.04 0.04 0.4"/></geometry>
+      <origin xyz="0 0 0.2" rpy="0 0 0"/>
+      <geometry><box size="0.04 0.04 0.4"/></geometry>
       <material name="yellow"/>
     </visual>
   </link>
-  <joint name="z_axis_joint" type="prismatic">
+  <joint name="arm_to_slider_joint" type="fixed">
     <parent link="sliding_module"/>
     <child link="vertical_arm"/>
     <origin rpy="0 0 0" xyz="0 0 0.03"/>
+  </joint>
+  <link name="lift_carriage">
+    <visual>
+      <geometry><box size="0.041 0.041 0.041"/></geometry>
+      <material name="red"/>
+    </visual>
+  </link>
+  <joint name="z_axis_lift_joint" type="prismatic">
+    <parent link="vertical_arm"/>
+    <child link="lift_carriage"/>
+    <origin xyz="0 0 0.05" rpy="0 0 0"/>
     <axis xyz="0 0 1"/>
-    <limit effort="100" lower="0.0" upper="0.4" velocity="1.0"/>
+    <limit lower="0.0" upper="0.35" effort="100" velocity="1.0"/>
   </joint>
   <link name="gripper_body">
     <visual>
+      <origin xyz="0 0.05 0" rpy="0 0 0"/>
       <geometry><box size="0.05 0.1 0.05"/></geometry>
       <material name="red"/>
@@ -44,7 +57,7 @@
   </link>
   <joint name="y_axis_forward_joint" type="prismatic">
-    <parent link="vertical_arm"/>
+    <parent link="lift_carriage"/>
     <child link="gripper_body"/>
-    <origin xyz="0 0.05 0.35" rpy="0 0 0"/>
+    <origin xyz="0 0.02 0" rpy="0 0 0"/>
     <axis xyz="0 1 0"/>
     <limit lower="0.0" upper="0.2" effort="100" velocity="1.0"/>

Commit message: update model

File: src/robot/kim_description/urdf/kim_kardashian.urdf.xacro (robot description, xacro)
@@ -5,38 +5,52 @@
   <material name="red"><color rgba="0.8 0 0 1"/></material>
   <material name="yellow"><color rgba="1 1 0 1"/></material>
+  <material name="green"><color rgba="0 0.8 0 1"/></material>
   <link name="base_link">
     <visual>
-      <geometry><box size="2.0 0.05 0.05"/></geometry>
-      <material name="grey"/>
+      <geometry><box size="0.05 0.3 0.02"/></geometry>
+      <material name="green"/>
     </visual>
   </link>
-  <link name="sliding_module">
+  <link name="x_rail_assembly">
     <visual>
-      <geometry><box size="0.15 0.15 0.06"/></geometry>
+      <geometry><box size="0.3 0.05 0.02"/></geometry>
+      <material name="blue"/>
+    </visual>
+  </link>
+  <joint name="y_axis_joint" type="prismatic">
+    <parent link="base_link"/>
+    <child link="x_rail_assembly"/>
+    <origin xyz="0 0 0.02" rpy="0 0 0"/>
+    <axis xyz="0 1 0"/>
+    <limit lower="-0.12" upper="0.12" effort="100" velocity="1.0"/>
+  </joint>
+  <link name="x_slider">
+    <visual>
+      <geometry><box size="0.06 0.06 0.02"/></geometry>
       <material name="blue"/>
     </visual>
   </link>
   <joint name="x_axis_joint" type="prismatic">
-    <parent link="base_link"/>
-    <child link="sliding_module"/>
-    <origin xyz="0 0 0.05" rpy="0 0 0"/>
+    <parent link="x_rail_assembly"/>
+    <child link="x_slider"/>
+    <origin xyz="0 0 0.02" rpy="0 0 0"/>
     <axis xyz="1 0 0"/>
-    <limit lower="-0.9" upper="0.9" effort="100" velocity="1.0"/>
+    <limit lower="-0.12" upper="0.12" effort="100" velocity="1.0"/>
   </joint>
   <link name="vertical_arm">
     <visual>
-      <origin xyz="0 0 0.2" rpy="0 0 0"/>
-      <geometry><box size="0.04 0.04 0.4"/></geometry>
+      <origin xyz="0 0 0.05" rpy="0 0 0"/>
+      <geometry><box size="0.03 0.03 0.1"/></geometry>
       <material name="yellow"/>
     </visual>
   </link>
-  <joint name="arm_to_slider_joint" type="fixed">
-    <parent link="sliding_module"/>
+  <joint name="arm_to_x_joint" type="fixed">
+    <parent link="x_slider"/>
     <child link="vertical_arm"/>
-    <origin rpy="0 0 0" xyz="0 0 0.03"/>
+    <origin xyz="0 0 0.01" rpy="0 0 0"/>
   </joint>
-  <link name="lift_carriage">
+  <link name="gripper_body">
     <visual>
-      <geometry><box size="0.041 0.041 0.041"/></geometry>
+      <geometry><box size="0.04 0.04 0.04"/></geometry>
       <material name="red"/>
     </visual>
@@ -44,35 +58,35 @@
   <joint name="z_axis_lift_joint" type="prismatic">
     <parent link="vertical_arm"/>
-    <child link="lift_carriage"/>
-    <origin xyz="0 0 0.05" rpy="0 0 0"/>
+    <child link="gripper_body"/>
+    <origin xyz="0 0.04 0.05" rpy="0 0 0"/>
     <axis xyz="0 0 1"/>
-    <limit lower="0.0" upper="0.35" effort="100" velocity="1.0"/>
-  </joint>
-  <link name="gripper_body">
-    <visual>
-      <origin xyz="0 0.05 0" rpy="0 0 0"/>
-      <geometry><box size="0.05 0.1 0.05"/></geometry>
-      <material name="red"/>
-    </visual>
-  </link>
-  <joint name="y_axis_forward_joint" type="prismatic">
-    <parent link="lift_carriage"/>
-    <child link="gripper_body"/>
-    <origin xyz="0 0.02 0" rpy="0 0 0"/>
-    <axis xyz="0 1 0"/>
-    <limit lower="0.0" upper="0.2" effort="100" velocity="1.0"/>
+    <limit lower="-0.04" upper="0.04" effort="100" velocity="1.0"/>
   </joint>
   <link name="finger_left">
     <visual>
-      <geometry><box size="0.01 0.05 0.02"/></geometry>
+      <geometry><box size="0.01 0.04 0.01"/></geometry>
       <material name="grey"/>
     </visual>
   </link>
-  <joint name="finger_joint" type="prismatic">
+  <joint name="finger_joint_left" type="prismatic">
     <parent link="gripper_body"/>
     <child link="finger_left"/>
-    <origin xyz="-0.02 0.1 0" rpy="0 0 0"/>
+    <origin xyz="-0.02 0.04 0" rpy="0 0 0"/>
     <axis xyz="1 0 0"/>
-    <limit lower="0" upper="0.02" effort="10" velocity="1.0"/>
+    <limit lower="-0.01" upper="0.01" effort="10" velocity="1.0"/>
+  </joint>
+  <link name="finger_right">
+    <visual>
+      <geometry><box size="0.01 0.04 0.01"/></geometry>
+      <material name="grey"/>
+    </visual>
+  </link>
+  <joint name="finger_joint_right" type="prismatic">
+    <parent link="gripper_body"/>
+    <child link="finger_right"/>
+    <origin xyz="0.02 0.04 0" rpy="0 0 0"/>
+    <axis xyz="1 0 0"/>
+    <limit lower="-0.01" upper="0.01" effort="10" velocity="1.0"/>
+    <mimic joint="finger_joint_left" multiplier="-1.0"/>
   </joint>
 </robot>
